File: arisu.kicad_pcb (KiCad board)
At the start: 2 copper layers, 339.1 x 118.7 mm, 176 parts, among them J1 USB_B_Micro, SW1 SW_Push, SW10 SW_Push, SW11 SW_Push, SW12 SW_Push, SW13 SW_Push, SW14 SW_Push, SW15 SW_Push, SW16 SW_Push, SW17 SW_Push, SW18 SW_Push, SW19 SW_Push, SW2 SW_Push, SW20 SW_Push, SW21 SW_Push, SW22 SW_Push, SW23 SW_Push, SW24 SW_Push, SW25 SW_Push, SW26 SW_Push, SW27 SW_Push, SW28 SW_Push, SW29 SW_Push, SW3 SW_Push, SW30 SW_Push, SW31 SW_Push, SW32 SW_Push, SW33 SW_Push, SW34 SW_Push, SW35 SW_Push, SW36 SW_Push, SW37 SW_Push, SW38 SW_Push, SW39 SW_Push, SW4 SW_Push, SW40 SW_Push, SW41 SW_Push, SW42 SW_Push, SW43 SW_Push, SW44 SW_Push, SW45 SW_Push, SW46 SW_Push, SW47 SW_Push, SW48 SW_Push, SW49 SW_Push, SW5 SW_Push, SW50 SW_Push, SW51 SW_Push, SW52 SW_Push, SW53 SW_Push, SW54 SW_Push, SW55 SW_Push, SW56 SW_Push, SW57 SW_Push, SW58 SW_Push, SW59 SW_Push, SW6 SW_Push, SW60 SW_Push, SW61 SW_Push, SW62 SW_Push, SW63 SW_Push, SW64 SW_Push, SW65 SW_Push, SW66 SW_Push, SW67 SW_Push, SW7 SW_Push, SW8 SW_Push, SW9 SW_Push, U1 USBLC6-2SC6, U2 ATmega32U4-AU, Y1 Crystal_GND24

Commit message: Finalize sch and pcb
Parts:
- removed G*** (x2): LOGO, arisu:arisu-logo
- removed PF4: PF4, Pin_Headers:Pin_Header_Straight_1x01_Pitch2.54mm
- added D68: D, Diodes_SMD:D_SOD-123, B.Cu at (-27.0, -1.19)
- added D69: D, Diodes_SMD:D_SOD-123, B.Cu at (-31.0, 17.9)
- added D70: D, Diodes_SMD:D_SOD-123, B.Cu at (-37.7, 36.9)
- added SW68: SW_Push, MX_Switch:SW_Cherry_MX_1.00u_PCB, F.Cu at (-32.9, -14.7)
- added SW69: SW_Push, MX_Switch:SW_Cherry_MX_1.00u_PCB, F.Cu at (-37.3, 4.37)
- added SW70: SW_Push, MX_Switch:SW_Cherry_MX_1.00u_PCB, F.Cu at (-44.1, 23.4)
- moved D51 61.2 mm to (215.0, 2.27)
- moved D66 61.2 mm to (304.4, 37.1)
- moved SW54 61.2 mm to (241.0, 47.6)
- moved D48 61.2 mm to (209.1, 23.7)
- moved D50 61.2 mm to (228.2, 60.9)
- moved D52 61.2 mm to (228.7, 22.8)
- moved D61 61.2 mm to (285.4, 65.7)
- moved D62 61.2 mm to (285.4, 84.7)
- moved D63 61.2 mm to (272.2, 3.77)
- moved D64 61.2 mm to (296.0, -0.99)
- moved D65 61.2 mm to (300.1, 18.1)
- moved D67 61.2 mm to (304.4, 84.7)
- moved H7 61.2 mm to (293.8, 4.76)
- moved H8 61.2 mm to (298.1, 71.4)
- moved SW49 61.2 mm to (212.4, 28.6)
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- renumbered PF6 to J10, PF7 to J11, VCC to J12, D+ to J13, D- to J14, GND to J15, MISO to J2, VCC to J3, SCK to J4, MOSI to J5, RES to J6, GND to J7, PF5 to J9
Connections:
- SW1 pad 1: /col0 -> /col1
- SW10 pad 1: /col2 -> /col3
- SW11 pad 1: /col2 -> /col3
- SW12 pad 1: /col2 -> /col3
- SW13 pad 1: /col2 -> /col3
- SW14 pad 1: /col2 -> /col3
- SW15 pad 1: /col3 -> /col4
- SW16 pad 1: /col3 -> /col4
- SW17 pad 1: /col3 -> /col4
- SW18 pad 1: /col3 -> /col4
- SW19 pad 1: /col4 -> /col5
- SW2 pad 1: /col0 -> /col1
- SW20 pad 1: /col4 -> /col5
- SW21 pad 1: /col4 -> /col5
- SW22 pad 1: /col4 -> /col5
- SW23 pad 1: /col4 -> /col5
- SW24 pad 1: /col5 -> /col6
- SW25 pad 1: /col5 -> /col6
- SW26 pad 1: /col5 -> /col6
- SW27 pad 1: /col5 -> /col6
- SW28 pad 1: /col5 -> /col6
- SW29 pad 1: /col6 -> /col7
- SW3 pad 1: /col0 -> /col1
- SW30 pad 1: /col6 -> /col7
- SW31 pad 1: /col6 -> /col7
- SW32 pad 1: /col6 -> /col7
- SW38 pad 1: /col8 -> /col9
- SW39 pad 1: /col8 -> /col9
- SW4 pad 1: /col0 -> /col1
- SW40 pad 1: /col8 -> /col9
- SW41 pad 1: /col8 -> /col9
- SW42 pad 1: /col9 -> /col10
- SW43 pad 1: /col9 -> /col10
- SW44 pad 1: /col9 -> /col10
- SW45 pad 1: /col9 -> /col10
- SW46 pad 1: /col9 -> /col10
- SW47 pad 1: /col10 -> /col11
- SW48 pad 1: /col10 -> /col11
- SW49 pad 1: /col10 -> /col11
- SW5 pad 1: /col0 -> /col1
- SW50 pad 1: /col10 -> /col11
- SW51 pad 1: /col11 -> /col12
- SW52 pad 1: /col11 -> /col12
- SW53 pad 1: /col11 -> /col12
- SW54 pad 1: /col11 -> /col12
- SW55 pad 1: /col12 -> /col13
- SW56 pad 1: /col12 -> /col13
- SW57 pad 1: /col12 -> /col13
- SW58 pad 1: /col12 -> /col13
- SW59 pad 1: /col13 -> /col14
- SW6 pad 1: /col1 -> /col2
- SW60 pad 1: /col13 -> /col14
- SW61 pad 1: /col13 -> /col14
- SW62 pad 1: /col13 -> /col14
- SW7 pad 1: /col1 -> /col2
- SW8 pad 1: /col1 -> /col2
- SW9 pad 1: /col1 -> /col2
- U2 pad 1: /col2 -> /col3
- U2 pad 12: /col9 -> /col10
- U2 pad 25: /col6 -> /col7
- U2 pad 26: /col13 -> /col14
- U2 pad 27: /col12 -> /col13
- U2 pad 28: /col11 -> /col12
- U2 pad 29: /col10 -> /col11
- U2 pad 30: /col5 -> /col6
- U2 pad 31: /col4 -> /col5
- U2 pad 32: /col3 -> /col4
- U2 pad 39: /PF4 -> /col0
- U2 pad 40: /col1 -> /col2
- U2 pad 41: /col0 -> /col1
- U2 pad 8: /col8 -> /col9
Routing:
- net /col14: track 0.00 -> 269.0 mm
- net /col8: track 104.4 -> 0.00 mm
- net /col7: track 0.00 -> 96.8 mm
- net /col10: track 221.3 -> 141.1 mm, vias 0 -> 2
- net /col3: track 133.3 -> 175.7 mm, vias 0 -> 2
- net /PF4: track 38.1 -> 0.00 mm, vias 1 -> 0
- net /col1: track 166.8 -> 204.4 mm
- net /col9: track 141.1 -> 104.4 mm, vias 2 -> 0
- net /row2: track 399.4 -> 434.8 mm
- net /row1: track 384.1 -> 414.5 mm
- net /row0: track 328.0 -> 353.8 mm
- net /col6: track 96.8 -> 121.5 mm
- net /col13: track 269.0 -> 249.0 mm
- net /col12: track 249.0 -> 230.6 mm
- net /col5: track 121.5 -> 135.2 mm
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Other:
- board size 339.1 x 118.7 mm -> 361.7 x 118.7 mm
