File: matrix.sch (KiCad schematic (older format))
At the start: 134 parts, among them SW1 SW_Push, SW10 SW_Push, SW11 SW_Push, SW12 SW_Push, SW13 SW_Push, SW14 SW_Push, SW15 SW_Push, SW16 SW_Push, SW17 SW_Push, SW18 SW_Push, SW19 SW_Push, SW2 SW_Push, SW20 SW_Push, SW21 SW_Push, SW22 SW_Push, SW23 SW_Push, SW24 SW_Push, SW25 SW_Push, SW26 SW_Push, SW27 SW_Push, SW28 SW_Push, SW29 SW_Push, SW3 SW_Push, SW30 SW_Push, SW31 SW_Push, SW32 SW_Push, SW33 SW_Push, SW34 SW_Push, SW35 SW_Push, SW36 SW_Push, SW37 SW_Push, SW38 SW_Push, SW39 SW_Push, SW4 SW_Push, SW40 SW_Push, SW41 SW_Push, SW42 SW_Push, SW43 SW_Push, SW44 SW_Push, SW45 SW_Push, SW46 SW_Push, SW47 SW_Push, SW48 SW_Push, SW49 SW_Push, SW5 SW_Push, SW50 SW_Push, SW51 SW_Push, SW52 SW_Push, SW53 SW_Push, SW54 SW_Push, SW55 SW_Push, SW56 SW_Push, SW57 SW_Push, SW58 SW_Push, SW59 SW_Push, SW6 SW_Push, SW60 SW_Push, SW61 SW_Push, SW62 SW_Push, SW63 SW_Push, SW64 SW_Push, SW65 SW_Push, SW66 SW_Push, SW67 SW_Push, SW7 SW_Push, SW8 SW_Push, SW9 SW_Push

Commit message: Finalize sch and pcb
Parts:
- added D68, D69, D70: D, Diodes_SMD:D_SOD-123, symbol Device:D
- added SW68, SW69, SW70: SW_Push, MX_Switch:SW_Cherry_MX_1.00u_PCB, symbol Switch:SW_Push
Connections:
- net col0: now also SW68.1, SW69.1, SW70.1; no longer SW1.1, SW2.1, SW3.1, SW4.1, SW5.1
- net col1: now also SW1.1, SW2.1, SW3.1, SW4.1, SW5.1; no longer SW6.1, SW7.1, SW8.1, SW9.1
- net col10: now also SW42.1, SW43.1, SW44.1, SW45.1, SW46.1; no longer SW47.1, SW48.1, SW49.1, SW50.1
- net col11: now also SW47.1, SW48.1, SW49.1, SW50.1; no longer SW51.1, SW52.1, SW53.1, SW54.1
- net col12: now also SW51.1, SW52.1, SW53.1, SW54.1; no longer SW55.1, SW56.1, SW57.1, SW58.1
- net col13: now also SW55.1, SW56.1, SW57.1, SW58.1; no longer SW59.1, SW60.1, SW61.1, SW62.1
- net col14: now also SW59.1, SW60.1, SW61.1, SW62.1; no longer SW63.1, SW64.1, SW65.1, SW66.1, SW67.1
- net col2: now also SW6.1, SW7.1, SW8.1, SW9.1; no longer SW10.1, SW11.1, SW12.1, SW13.1, SW14.1
- net col3: now also SW10.1, SW11.1, SW12.1, SW13.1, SW14.1; no longer SW15.1, SW16.1, SW17.1, SW18.1
- net col4: now also SW15.1, SW16.1, SW17.1, SW18.1; no longer SW19.1, SW20.1, SW21.1, SW22.1, SW23.1
- net col5: now also SW19.1, SW20.1, SW21.1, SW22.1, SW23.1; no longer SW24.1, SW25.1, SW26.1, SW27.1, SW28.1
- net col6: now also SW24.1, SW25.1, SW26.1, SW27.1, SW28.1; no longer SW29.1, SW30.1, SW31.1, SW32.1
- net col7: now also SW29.1, SW30.1, SW31.1, SW32.1; no longer SW33.1, SW34.1, SW35.1, SW36.1, SW37.1
- net col8: now also SW33.1, SW34.1, SW35.1, SW36.1, SW37.1; no longer SW38.1, SW39.1, SW40.1, SW41.1
- net col9: now also SW38.1, SW39.1, SW40.1, SW41.1; no longer SW42.1, SW43.1, SW44.1, SW45.1, SW46.1
- net row0: now also D68.1 (K)
- net row1: now also D69.1 (K)
- net row2: now also D70.1 (K)
- new net: D68.2 (A), SW68.2
- new net: D69.2 (A), SW69.2
- new net: D70.2 (A), SW70.2
- new net col15: SW63.1, SW64.1, SW65.1, SW66.1, SW67.1
Other:
- note added: "LM1"
- note added: "LM2"
- note added: "LM3"
Changed lines of the file:
@@
 EESchema Schematic File Version 4
+LIBS:arisu-cache
 EELAYER 30 0
 EELAYER END
@@
 Text HLabel 950  1950 0    50   3State ~ 0
 row0
+Text HLabel 1200 750  1    50   3State ~ 0
+col1
 Text HLabel 1850 750  1    50   3State ~ 0
-col1
-Text HLabel 2500 750  1    50   3State ~ 0
 col2
 Text HLabel 950  2950 0    50   3State ~ 0
@@
 	1    0    0    -1
 $EndComp
-Text HLabel 1200 750  1    50   3State ~ 0
+Text HLabel 600  750  1    50   3State ~ 0
 col0
+Text HLabel 2500 750  1    50   3State ~ 0
+col3
 Text HLabel 3150 750  1    50   3State ~ 0
-col3
+col4
 Text HLabel 3800 750  1    50   3State ~ 0
-col4
+col5
 Text HLabel 4450 750  1    50   3State ~ 0
-col5
+col6
 Text HLabel 5100 750  1    50   3State ~ 0
-col6
+col7
 Text HLabel 5750 750  1    50   3State ~ 0
-col7
+col8
 Text HLabel 6400 750  1    50   3State ~ 0
-col8
+col9
 Text HLabel 7050 750  1    50   3State ~ 0
-col9
+col10
 Text HLabel 7700 750  1    50   3State ~ 0
-col10
+col11
 Text HLabel 8350 750  1    50   3State ~ 0
-col11
+col12
 Text HLabel 9000 750  1    50   3State ~ 0
-col12
+col13
 Text HLabel 9650 750  1    50   3State ~ 0
-col13
-Text HLabel 10300 750  1    50   3State ~ 0
 col14
 $Comp
@@
 $EndComp
 Wire Wire Line
-	950  1950 1600 1950
-Wire Wire Line
-	950  2950 1600 2950
+	950  1950 1000 1950
+Wire Wire Line
+	950  2950 1000 2950
 $Comp
 L Switch:SW_Push SW2
@@
 $EndComp
 Wire Wire Line
-	950  3950 1600 3950
+	950  3950 1000 3950
 Wire Wire Line
 	950  4950 1600 4950
@@
 Wire Wire Line
 	1600 5950 2900 5950
+$Comp
+L Switch:SW_Push SW68
+U 1 1 60923016
+P 800 1600
+F 0 "SW68" H 800 1885 50  0000 C CNN
+F 1 "SW_Push" H 800 1794 50  0000 C CNN
+F 2 "MX_Switch:SW_Cherry_MX_1.00u_PCB" H 800 1800 50  0001 C CNN
+F 3 "" H 800 1800 50  0001 C CNN
+	1    800  1600
+	1    0    0    -1
+$EndComp
+$Comp
+L Device:D D68
+U 1 1 6092301C
+P 1000 1750
+F 0 "D68" V 1050 1950 50  0000 R CNN
+F 1 "D" V 950 1900 50  0000 R CNN
+F 2 "Diodes_SMD:D_SOD-123" H 1000 1750 50  0001 C CNN
+F 3 "~" H 1000 1750 50  0001 C CNN
+	1    1000 1750
+	0    -1   -1   0
+$EndComp
+Connection ~ 600  1600
+Wire Wire Line
+	600  750  600  1600
+Wire Wire Line
+	600  1600 600  2600
+Text Notes 750  1200 0    100  ~ 0
+LM1
+$Comp
+L Switch:SW_Push SW69
+U 1 1 6092D432
+P 800 2600
+F 0 "SW69" H 800 2885 50  0000 C CNN
+F 1 "SW_Push" H 800 2794 50  0000 C CNN
+F 2 "MX_Switch:SW_Cherry_MX_1.00u_PCB" H 800 2800 50  0001 C CNN
+F 3 "" H 800 2800 50  0001 C CNN
+	1    800  2600
+	1    0    0    -1
+$EndComp
+$Comp
+L Device:D D69
+U 1 1 6092D438
+P 1000 2750
+F 0 "D69" V 1050 2950 50  0000 R CNN
+F 1 "D" V 950 2900 50  0000 R CNN
+F 2 "Diodes_SMD:D_SOD-123" H 1000 2750 50  0001 C CNN
+F 3 "~" H 1000 2750 50  0001 C CNN
+	1    1000 2750
+	0    -1   -1   0
+$EndComp
+Connection ~ 600  2600
+Wire Wire Line
+	600  1750 600  2600
+Text Notes 750  2200 0    100  ~ 0
+LM2
+$Comp
+L Switch:SW_Push SW70
+U 1 1 609384E4
+P 800 3600
+F 0 "SW70" H 800 3885 50  0000 C CNN
+F 1 "SW_Push" H 800 3794 50  0000 C CNN
+F 2 "MX_Switch:SW_Cherry_MX_1.00u_PCB" H 800 3800 50  0001 C CNN
+F 3 "" H 800 3800 50  0001 C CNN
+	1    800  3600
+	1    0    0    -1
+$EndComp
+$Comp
+L Device:D D70
+U 1 1 609384EA
+P 1000 3750
+F 0 "D70" V 1050 3950 50  0000 R CNN
+F 1 "D" V 950 3900 50  0000 R CNN
+F 2 "Diodes_SMD:D_SOD-123" H 1000 3750 50  0001 C CNN
+F 3 "~" H 1000 3750 50  0001 C CNN
+	1    1000 3750
+	0    -1   -1   0
+$EndComp
+Text Notes 750  3200 0    100  ~ 0
+LM3
+Text HLabel 10300 750  1    50   3State ~ 0
+col15
+Wire Wire Line
+	1000 1900 1000 1950
+Connection ~ 1000 1950
+Wire Wire Line
+	1000 1950 1600 1950
+Wire Wire Line
+	1000 2900 1000 2950
+Connection ~ 1000 2950
+Wire Wire Line
+	1000 2950 1600 2950
+Wire Wire Line
+	1000 3900 1000 3950
+Connection ~ 1000 3950
+Wire Wire Line
+	1000 3950 1600 3950
+Wire Wire Line
+	600  2600 600  3600
 $EndSCHEMATC
